File: Gaus-Beschleuniger.kicad_pcb (KiCad board)
At the start: 2 copper layers, 121 parts, among them J1 Conn_01x02, J10 Conn_01x04, J11 Conn_01x03, J12 Conn_01x04_Socket, J13 Conn_01x03, J2 Conn_01x02, J3 Conn_01x02, J4 Conn_01x02, J5 Conn_01x02, J6 Conn_01x02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

Commit message: start layout
Parts:
- removed D23: D_Schottky, Diode_SMD:D_SOD-123
- removed R21, R22: 10k, Resistor_SMD:R_0805_2012Metric_Pad1.20x1.40mm_HandSolder
- added C26: 1000pF, Capacitor_SMD:C_1206_3216Metric_Pad1.33x1.80mm_HandSolder, F.Cu at (202.5, -17.0)
- added REF**: MountingHole_3.2mm_M3_DIN965, MountingHole:MountingHole_3.2mm_M3_DIN965, F.Cu at (287.5, 140.0)
- added REF**: MountingHole_3.2mm_M3_DIN965, MountingHole:MountingHole_3.2mm_M3_DIN965, F.Cu at (152.5, 160.0)
- added REF**: MountingHole_3.2mm_M3_DIN965, MountingHole:MountingHole_3.2mm_M3_DIN965, F.Cu at (287.5, 160.0)
- added REF**: MountingHole_3.2mm_M3_DIN965, MountingHole:MountingHole_3.2mm_M3_DIN965, F.Cu at (152.5, 140.0)
- D15, D4: footprint Package_TO_SOT_THT:TO-247-3_Vertical -> Package_TO_SOT_THT:TO-247-3_Horizontal_TabDown; moved to B.Cu
- Q3, Q4, Q5, Q6: footprint LED_THT:LED_SideEmitter_Rectangular_W4.5mm_H1.6mm -> OptoDevice:Osram_LPT80A
- TR1: moved to F.Cu
- moved R20 199.6 mm to (131.0, 140.0), turned to 180 degrees
- moved R5 178.9 mm to (168.0, 142.5), turned to 0 degrees
- moved R11 177.9 mm to (168.0, 158.0), turned to 0 degrees
- moved D7 169.9 mm to (171.7, 142.5)
- moved D6 169.3 mm to (173.8, 163.5)
- moved Q3 168.9 mm to (171.7, 157.9), turned to 90 degrees
- moved R14 150.6 mm to (230.0, 142.5), turned to 0 degrees
- moved R15 149.3 mm to (230.0, 158.0), turned to 0 degrees
- moved D8 148.9 mm to (210.7, 142.5)
- moved R12 148.9 mm to (217.0, 142.5)
- moved Q4 147.6 mm to (210.7, 157.9), turned to 90 degrees
- moved R13 147.6 mm to (217.0, 158.0)
- moved D9 147.2 mm to (213.8, 163.5)
- moved D10 142.0 mm to (233.7, 142.5)
- moved D11 140.9 mm to (235.8, 163.5)
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Connections:
- D24 pad 1: Net-(D24-K) -> /Firing-Stage/discharge_gate
- J4 pad 1: /Firing-Stage/HV_S1 -> /Firing-Stage/HV_S2
- J4 pad 2: /Firing-Stage/HV_S1 -> /Firing-Stage/HV_S2
- Q1 pad 1: Net-(D24-K) -> /Firing-Stage/discharge_gate
- Q2 pad 1: Net-(D23-K) -> /Firing-Stage/discharge_gate
- R6 pad 1: Net-(D24-K) -> /Firing-Stage/discharge_gate
- R7 pad 2: Net-(D24-K) -> /Firing-Stage/discharge_gate
Routing:
- net /Firing-Stage/HV_S1: track 0.00 -> 72.3 mm, vias 0 -> 2
- net /Firing-Stage/HV_S2: track 0.00 -> 72.0 mm
- net +5V: track 0.00 -> 62.0 mm
- net /Firing-Stage/discharge_gate: track 0.00 -> 35.5 mm
- net /Controller/Discharge: track 0.00 -> 33.6 mm
- net /Controller/Stage1_optical2: track 0.00 -> 13.3 mm
- net /Controller/Stage2_optical2: track 0.00 -> 13.3 mm
- net Net-(Q1-D): track 0.00 -> 10.2 mm
- net Net-(Q2-D): track 0.00 -> 9.98 mm
- net /Controller/Stage2_optical1: track 0.00 -> 8.53 mm
- net /Controller/Stage1_optical1: track 0.00 -> 8.53 mm
- net Net-(D7-A): track 0.00 -> 7.81 mm
- net Net-(D10-A): track 0.00 -> 7.81 mm
- net /Controller/uC_Discharge: track 0.00 -> 5.47 mm
- net Net-(Q9-D-Pad5): track 0.00 -> 5.24 mm
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- added copper zone on F.Cu, net /Cap-Charger/HV-Charger_out
- added copper zone on F.Cu, net /Firing-Stage/HV_S1
- added copper zone on F.Cu, net /Firing-Stage/HV_S2
Other:
- board text added: "GND HV1"
- board text added: "HV2 GND"

Commit message: layout weiter
Parts:
- removed the REF** at (287.5, 140.0)
- removed the REF** at (287.5, 160.0)
- added REF**: MountingHole_3.2mm_M3_DIN965, MountingHole:MountingHole_3.2mm_M3_DIN965, F.Cu at (287.5, 160.5)
- added REF**: MountingHole_3.2mm_M3_DIN965, MountingHole:MountingHole_3.2mm_M3_DIN965, F.Cu at (287.5, 139.5)
- moved R20 92.8 mm to (223.2, 150.0), turned to -90 degrees
- moved C16 92.0 mm to (133.0, 64.0)
- moved C17 92.0 mm to (133.0, 67.3)
- moved C18 92.0 mm to (133.0, 70.7)
- moved C19 92.0 mm to (129.0, 78.0)
- moved C20 92.0 mm to (129.0, 81.3)
- moved C21 92.0 mm to (129.0, 84.7)
- moved C22 92.0 mm to (138.0, 70.0)
- moved C23 92.0 mm to (144.7, 67.0)
- moved C24 92.0 mm to (144.7, 58.0)
- moved C26 92.0 mm to (183.5, 73.0)
- moved D16 92.0 mm to (174.5, 69.5)
- moved D18 92.0 mm to (85.9, 76.0)
- moved D3 92.0 mm to (107.5, 79.3)
- moved J8 92.0 mm to (181.5, 67.3)
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Connections:
- net Net-(D15-A) renamed /Firing-Stage/S2_D
- net Net-(D4-A) renamed /Firing-Stage/S1_D
Routing:
- net +5V: track 62.0 -> 218.6 mm, vias 0 -> 2
- net /Controller/Stage2_optical2: track 13.3 -> 114.5 mm
- net /Controller/Stage1_trigger_lp: track 0.00 -> 52.7 mm
- net /Controller/Stage2_trigger_lp: track 0.00 -> 44.5 mm
- net /Controller/Stage2_charge_sense: track 0.00 -> 36.0 mm
- net /Controller/Discharge: track 33.6 -> 0.00 mm
- net /Controller/Stage2_optical1: track 8.53 -> 39.6 mm
- net /Controller/Stage1_optical1: track 8.53 -> 37.4 mm
- net /Firing-Stage/discharge_gate: track 35.5 -> 13.9 mm
- net /Controller/Stage1_charge_sense: track 0.00 -> 18.9 mm
- net /Controller/Stage1_optical2: track 13.3 -> 30.0 mm
- net Net-(Q2-D): track 9.98 -> 17.2 mm
- net Net-(Q1-D): track 10.2 -> 17.2 mm
- net /Controller/uC_Discharge: track 5.47 -> 0.00 mm
- net Net-(R4-Pad1): track 0.00 -> 3.31 mm
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- added copper zone on F.Cu, net /Firing-Stage/S1_D
- added copper zone on F.Cu, net /Firing-Stage/S2_D
- added copper zone on B.Cu, net GND

Commit message: firing routing, uC routing done
Parts:
- moved R37 99.7 mm to (127.5, 138.0), turned to -90 degrees
- moved R39 98.3 mm to (125.0, 138.0), turned to -90 degrees
- moved R40 96.5 mm to (122.5, 138.0), turned to 90 degrees
- moved SW6 94.2 mm to (116.8, 199.2)
- moved R41 93.3 mm to (120.0, 184.5)
- moved R36 90.8 mm to (119.0, 160.5), turned to 180 degrees
- moved SW5 85.4 mm to (101.8, 199.2)
- moved R35 85.0 mm to (105.0, 184.5)
- moved R33 83.5 mm to (110.0, 160.5)
- moved SW4 79.4 mm to (86.8, 199.2)
- moved D22 79.3 mm to (120.0, 178.7), turned to -90 degrees
- moved C25 76.7 mm to (114.2, 167.7), turned to 90 degrees
- moved R38 76.3 mm to (105.0, 160.5), turned to 180 degrees
- moved A1 74.8 mm to (124.0, 141.9), turned to -90 degrees
- moved R34 73.7 mm to (90.0, 185.0)
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Routing:
- net +5V: track 218.6 -> 507.9 mm, vias 2 -> 10
- net /Controller/Stage2_optical1: track 39.6 -> 239.3 mm, vias 0 -> 6
- net /Controller/Discharge: track 0.00 -> 198.6 mm, vias 0 -> 2
- net /Controller/Stage1_optical2: track 30.0 -> 223.8 mm, vias 0 -> 4
- net /Controller/Stage2_charge_sense: track 36.0 -> 225.7 mm, vias 0 -> 4
- net /Controller/Stage2_optical2: track 114.5 -> 295.3 mm, vias 0 -> 2
- net /Controller/uC_Discharge: track 0.00 -> 176.4 mm, vias 0 -> 2
- net /Controller/Stage2_trigger_lp: track 44.5 -> 198.7 mm, vias 0 -> 7
- net /Controller/uC_Charge: track 0.00 -> 131.0 mm, vias 0 -> 2
- net /Controller/uC_Stage2_trigger: track 0.00 -> 101.7 mm, vias 0 -> 4
- net /Controller/uC_trigger_in: track 0.00 -> 97.9 mm, vias 0 -> 2
- net /Controller/uC_Stage1_trigger: track 0.00 -> 81.2 mm, vias 0 -> 2
- net /Controller/Stage1_charge_sense: track 18.9 -> 96.4 mm, vias 0 -> 2
- net /Controller/Stage1_optical1: track 37.4 -> 105.5 mm, vias 0 -> 2
- net /Cap-Charger/EN: track 0.00 -> 65.4 mm, vias 0 -> 2
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- added copper zone on F.Cu, net +24V
- added copper zone on F.Cu, net +5V
- added copper zone on F.Cu, net Net-(D1-A1)
- added copper zone on F.Cu, net Net-(U1-CB)
- added copper zone on F.Cu, net Net-(U1-SW)
Other:
- board text added: "1"
- board text added: "Charge"
- board text added: "Charge Source: 1-2: uC 2-3: manuell"
- board text added: "Stage 1 Trigger: 1-2: uC 2-3: manuell 3-4: manuell routed to uC"
- board text added: "Stage 2 Trigger: 1-2: uC 2-3: manuell"
- board text added: "Trigger 1"
- board text added: "Trigger 2"

Commit message: placement and routing done drc errors, stiching vias and polish next
Parts:
- added BT1: Battery, Connector_AMASS:AMASS_XT60-M_1x02_P7.20mm_Vertical, B.Cu at (57.5, 113.6)
- moved D18 64.5 mm to (95.1, 110.0), turned to 180 degrees
- moved J9 55.5 mm to (85.0, 104.0), turned to 90 degrees
- moved D3 50.3 mm to (103.3, 105.5), turned to 180 degrees
- moved R30 46.7 mm to (96.5, 105.5), turned to 0 degrees
- moved C16 38.8 mm to (113.5, 108.2)
- moved R31 38.7 mm to (101.2, 117.0), turned to -90 degrees
- moved J8 36.1 mm to (158.2, 90.8), turned to 90 degrees
- moved C26 34.2 mm to (150.0, 108.5), turned to -90 degrees
- moved TR1 34.2 mm to (135.0, 107.5)
- moved R29 33.8 mm to (121.2, 112.5)
- moved C19 33.6 mm to (109.2, 117.0), turned to -90 degrees
- moved R27 33.5 mm to (121.2, 114.2)
- moved C24 33.5 mm to (120.0, 96.1), turned to -90 degrees
- moved Q9 33.3 mm to (119.5, 118.2)
- moved C22 32.8 mm to (119.8, 108.2), turned to 90 degrees
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Routing:
- net +5V: track 507.9 -> 662.2 mm, vias 10 -> 12
- net /Cap-Charger/EN: track 65.4 -> 137.9 mm
- net /Cap-Charger/~{DONE}: track 0.00 -> 62.7 mm, vias 0 -> 6
- net /Cap-Charger/Charge supply: track 16.4 -> 59.5 mm, vias 0 -> 2
- net Net-(D18-A): track 0.00 -> 36.2 mm, vias 0 -> 2
- net /Cap-Charger/HV-Charger_out: track 0.00 -> 12.9 mm
- net Net-(D18-K): track 0.00 -> 10.5 mm
- net Net-(U2-RBG): track 0.00 -> 5.70 mm
- net Net-(Q9-D-Pad5): track 5.24 -> 0.00 mm
- net Net-(D3-A): track 0.00 -> 3.23 mm
- net Net-(U2-RDCM): track 3.68 -> 5.66 mm
- net Net-(Q9-G): track 9.80 -> 11.1 mm
- net Net-(U2-RVout): track 3.89 -> 5.14 mm
- net /Controller/Discharge: track 198.6 -> 198.8 mm, vias 2 -> 0
- added copper zone on F.Cu, net /Cap-Charger/Charge supply
- added copper zone on F.Cu, net GND
- added copper zone on F.Cu, net Net-(D16-A)
- added copper zone on F.Cu, net Net-(D18-A)
- added copper zone on F.Cu, net Net-(Q9-D-Pad5)
- added copper zone on F.Cu, net Net-(U2-SOURCE)
Other:
- board text added: "Charged up!"
- board text added: "Vgate Source: 1-2: Vin-6V 2-3: Vin"

Commit message: Layout finished
Parts:
- removed REF** (x4): MountingHole_3.2mm_M3_DIN965, MountingHole:MountingHole_3.2mm_M3_DIN965
- added H1: MountingHole, MountingHole:MountingHole_4.3mm_M4_DIN965, F.Cu at (55.0, 90.0)
- added H2: MountingHole, MountingHole:MountingHole_4.3mm_M4_DIN965, F.Cu at (55.0, 210.0)
- added H3: MountingHole, MountingHole:MountingHole_4.3mm_M4_DIN965, F.Cu at (290.0, 90.0)
- added H4: MountingHole, MountingHole:MountingHole_4.3mm_M4_DIN965, F.Cu at (290.0, 210.0)
- added H5: MountingHole, MountingHole:MountingHole_3.2mm_M3_DIN965, F.Cu at (152.5, 139.5)
- added H6: MountingHole, MountingHole:MountingHole_3.2mm_M3_DIN965, F.Cu at (152.5, 160.5)
- added H7: MountingHole, MountingHole:MountingHole_3.2mm_M3_DIN965, F.Cu at (287.5, 139.5)
- added H8: MountingHole, MountingHole:MountingHole_3.2mm_M3_DIN965, F.Cu at (287.5, 160.5)
- moved J7 5.12 mm to (57.1, 122.5), turned to -90 degrees
- moved R31 0.50 mm to (101.2, 117.5)
Connections:
- J7 pad 1: GND -> Net-(BT1-+)
- J7 pad 2: Net-(BT1-+) -> GND
Routing:
- net Net-(U2-SOURCE): track 0.00 -> 4.45 mm
- net /Controller/uC_trigger_in: track 97.9 -> 97.4 mm
- net /Controller/Discharge: track 198.8 -> 198.3 mm
- net GND: vias 0 -> 465
- net /Controller/Stage2_trigger_lp: vias 7 -> 6
Other:
- board outline added: 245 x 130 mm
- board text added: "+5V GND nc HV"
- board text added: "5V"
- board text added: "GND +5V SCL SDA"
- board text added: "Gauss-Beschleuniger v0.1.0 Vin: 12-24 V"
- board text added: "VIN GND"
- board text added: "Vgate Source: 1-2: Vin 2-3: Vin-6V"
- board text removed: "Vgate Source: 1-2: Vin-6V 2-3: Vin"
