File: Gaus-Beschleuniger.kicad_pcb (KiCad board)
At the start: 2 copper layers, 245 x 130 mm, 128 parts, among them J1 Conn_01x02, J10 Conn_01x04, J11 Conn_01x03, J12 Conn_01x04_Socket, J13 Conn_01x03, J2 Conn_01x02, J3 Conn_01x02, J4 Conn_01x02, J5 Conn_01x02, J6 Conn_01x02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

Commit message: update fab files ;/
Parts:
- D16: value 1000V -> US2M_HF
- R23, R8: value 2k 5W SQP10AJB-2K -> 2k
- U2: value ~ -> LT3750
