File: 5V_Buck.kicad_sch (KiCad schematic)
At the start: 13 parts, among them U1 LMR50410

Commit message: update fab files ;/
Parts:
- C10, C11, C12: LCSC_Part_# (none) -> C13832
- C13, C9: LCSC_Part_# (none) -> C28233
- C14, C15: LCSC_Part_# (none) -> C441864
- L1: LCSC_Part_# (none) -> C3224592
- R1: LCSC_Part_# (none) -> C84376
- R2: LCSC_Part_# (none) -> C273823
- R25: LCSC_Part_# (none) -> C228640
- U1: LCSC_Part_# (none) -> C2841056; MPN LMR50410XFDBVR -> LMR50410XDBVR
Changed lines of the file:
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@@
 			)
 		)
-		(property "MPN" "LMR50410XFDBVR"
+		(property "MPN" " LMR50410XDBVR"
+			(at 76.2 46.99 0)
+			(effects
+				(font
+					(size 1.27 1.27)
+				)
+				(hide yes)
+			)
+		)
+		(property "LCSC_Part_#" "C2841056"
 			(at 76.2 46.99 0)
 			(effects
@@
 		)
 		(property "Voltage" "100V"
+			(at 33.02 46.99 0)
+			(effects
+				(font
+					(size 1.27 1.27)
+				)
+				(hide yes)
+			)
+		)
+		(property "LCSC_Part_#" "C13832"
 			(at 33.02 46.99 0)
 			(effects
@@
 			)
 		)
+		(property "LCSC_Part_#" "C273823"
+			(at 109.22 53.34 0)
+			(effects
+				(font
+					(size 1.27 1.27)
+				)
+				(hide yes)
+			)
+		)
 		(pin "1"
 		)
@@
 			)
 		)
+		(property "LCSC_Part_#" "C3224592"
+			(at 102.87 46.99 90)
+			(effects
+				(font
+					(size 1.27 1.27)
+				)
+				(hide yes)
+			)
+		)
 		(pin "1"
 		)
@@
 			)
 		)
+		(property "LCSC_Part_#" "C13832"
+			(at 45.72 46.99 0)
+			(effects
+				(font
+					(size 1.27 1.27)
+				)
+				(hide yes)
+			)
+		)
 		(pin "1"
 		)
@@
 			)
 		)
+		(property "LCSC_Part_#" "C13832"
+			(at 39.37 46.99 0)
+			(effects
+				(font
+					(size 1.27 1.27)
+				)
+				(hide yes)
+			)
+		)
 		(pin "1"
 		)
@@
 			)
 		)
+		(property "LCSC_Part_#" "C28233"
+			(at 52.07 46.99 0)
+			(effects
+				(font
+					(size 1.27 1.27)
+				)
+				(hide yes)
+			)
+		)
 		(pin "1"
 		)
@@
 			)
 		)
+		(property "LCSC_Part_#" "C228640"
+			(at 109.22 63.5 0)
+			(effects
+				(font
+					(size 1.27 1.27)
+				)
+				(hide yes)
+			)
+		)
 		(pin "2"
 		)
@@
 		)
 		(property "Voltage" "100V"
+			(at 91.44 44.45 0)
+			(effects
+				(font
+					(size 1.27 1.27)
+				)
+				(hide yes)
+			)
+		)
+		(property "LCSC_Part_#" "C28233"
 			(at 91.44 44.45 0)
 			(effects
@@
 			)
 		)
+		(property "LCSC_Part_#" ""
+			(at 133.35 63.5 90)
+			(effects
+				(font
+					(size 1.27 1.27)
+				)
+				(hide yes)
+			)
+		)
 		(pin "1"
 		)
@@
 		)
 		(property "Voltage" "10V"
+			(at 125.73 58.42 0)
+			(effects
+				(font
+					(size 1.27 1.27)
+				)
+				(hide yes)
+			)
+		)
+		(property "LCSC_Part_#" "C441864"
 			(at 125.73 58.42 0)
 			(effects
@@
 			)
 		)
+		(property "LCSC_Part_#" "C84376"
+			(at 133.35 54.61 0)
+			(effects
+				(font
+					(size 1.27 1.27)
+				)
+				(hide yes)
+			)
+		)
 		(pin "2"
 		)
@@
 			(at 118.11 58.42 0)
 			(effects
+				(font
+					(size 1.27 1.27)
+				)
+				(hide yes)
+			)
+		)
+		(property "LCSC_Part_#" "C441864"
+			(at 118.11 58.42 0)
+			(effects
