File: Cap-Charger.kicad_sch (KiCad schematic)
At the start: 23 parts, among them J8 Conn_01x04, J9 Conn_01x03, Q9 IRF7493

Commit message: rough placement
Parts:
- R27: footprint Resistor_SMD:R_0805_2012Metric_Pad1.20x1.40mm_HandSolder -> Resistor_SMD:R_0603_1608Metric_Pad0.98x0.95mm_HandSolder; MPN RC0805FR-0743KL -> RC0603FR-0743KL
- R29: footprint Resistor_SMD:R_0805_2012Metric_Pad1.20x1.40mm_HandSolder -> Resistor_SMD:R_0603_1608Metric_Pad0.98x0.95mm_HandSolder; MPN RC0805FR-0760K4L -> RC0603FR-0760K4L
- R30: value 20k0 -> 10k; MPN RC0805FR-0720KL -> RC0805FR-0710KL
- R31: MPN (none) -> RC0805FR-0710KL
Connections:
- net +5V: now also R30.1; no longer R30.2
- net at D3.2 (A): now also R30.2; no longer R30.1
Changed lines of the file:
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@@
+	)
+	(symbol
+		(lib_id "Device:R")
+		(at 86.36 87.63 90)
+		(unit 1)
+		(exclude_from_sim no)
+		(in_bom yes)
+		(on_board yes)
+		(dnp no)
+		(property "Reference" "R30"
+			(at 86.36 90.17 90)
+			(effects
+				(font
+					(size 1.27 1.27)
+				)
+			)
+		)
+		(property "Value" "10k"
+			(at 86.36 85.09 90)
+			(effects
+				(font
+					(size 1.27 1.27)
+				)
+			)
+		)
+		(property "Footprint" "Resistor_SMD:R_0805_2012Metric_Pad1.20x1.40mm_HandSolder"
+			(at 86.36 89.408 90)
+			(effects
+				(font
+					(size 1.27 1.27)
+				)
+				(hide yes)
+			)
+		)
+		(property "Datasheet" "~"
+			(at 86.36 87.63 0)
+			(effects
+				(font
+					(size 1.27 1.27)
+				)
+				(hide yes)
+			)
+		)
+		(property "Description" "Resistor"
+			(at 86.36 87.63 0)
+			(effects
+				(font
+					(size 1.27 1.27)
+				)
+				(hide yes)
+			)
+		)
+		(property "MPN" "RC0805FR-0710KL"
+			(at 86.36 87.63 90)
+			(effects
+				(font
+					(size 1.27 1.27)
+				)
+				(hide yes)
+			)
+		)
+		(pin "2"
+		)
+		(pin "1"
+		)
+		(instances
+			(project "Gaus-Beschleuniger"
+				(path "/10afecde-cced-4b16-9a8f-ba25affe517e/89601b47-33d3-45bd-90a7-6d36528e5bd8"
+					(reference "R30")
+					(unit 1)
+				)
+			)
+		)
 	)
 	(symbol
@@
 		(pin "1"
 		)
+		(pin "3"
+		)
+		(pin "8"
+		)
+		(pin "9"
+		)
 		(instances
 			(project ""
@@
 			)
 		)
+		(property "MPN" "RC0805FR-0710KL"
+			(at 99.06 100.33 0)
+			(effects
+				(font
+					(size 1.27 1.27)
+				)
+				(hide yes)
+			)
+		)
 		(pin "2"
 		)
@@
 			)
 		)
-		(property "Footprint" "Resistor_SMD:R_0805_2012Metric_Pad1.20x1.40mm_HandSolder"
+		(property "Footprint" "Resistor_SMD:R_0603_1608Metric_Pad0.98x0.95mm_HandSolder"
 			(at 143.51 79.248 90)
 			(effects
@@
 			)
 		)
-		(property "MPN" "RC0805FR-0760K4L"
+		(property "MPN" "RC0603FR-0760K4L"
 			(at 143.51 77.47 0)
 			(effects
@@
 				(path "/10afecde-cced-4b16-9a8f-ba25affe517e/89601b47-33d3-45bd-90a7-6d36528e5bd8"
 					(reference "R29")
-					(unit 1)
-				)
-			)
-		)
-	)
-	(symbol
-		(lib_id "Device:R")
-		(at 86.36 87.63 270)
-		(unit 1)
-		(exclude_from_sim no)
-		(in_bom yes)
-		(on_board yes)
-		(dnp no)
-		(property "Reference" "R30"
-			(at 86.36 90.17 90)
-			(effects
-				(font
-					(size 1.27 1.27)
-				)
-			)
-		)
-		(property "Value" "20k0"
-			(at 86.36 85.09 90)
-			(effects
-				(font
-					(size 1.27 1.27)
-				)
-			)
-		)
-		(property "Footprint" "Resistor_SMD:R_0805_2012Metric_Pad1.20x1.40mm_HandSolder"
-			(at 86.36 85.852 90)
-			(effects
-				(font
-					(size 1.27 1.27)
-				)
-				(hide yes)
-			)
-		)
-		(property "Datasheet" "~"
-			(at 86.36 87.63 0)
-			(effects
-				(font
-					(size 1.27 1.27)
-				)
-				(hide yes)
-			)
-		)
-		(property "Description" "Resistor"
-			(at 86.36 87.63 0)
-			(effects
-				(font
-					(size 1.27 1.27)
-				)
-				(hide yes)
-			)
-		)
-		(property "MPN" "RC0805FR-0720KL"
-			(at 86.36 87.63 0)
-			(effects
-				(font
-					(size 1.27 1.27)
-				)
-				(hide yes)
-			)
-		)
-		(pin "1"
-		)
-		(pin "2"
-		)
-		(instances
-			(project "Gaus-Beschleuniger"
-				(path "/10afecde-cced-4b16-9a8f-ba25affe517e/89601b47-33d3-45bd-90a7-6d36528e5bd8"
-					(reference "R30")
 					(unit 1)
 				)
@@
 			)
 		)
-		(property "Footprint" "Resistor_SMD:R_0805_2012Metric_Pad1.20x1.40mm_HandSolder"
+		(property "Footprint" "Resistor_SMD:R_0603_1608Metric_Pad0.98x0.95mm_HandSolder"
 			(at 135.89 84.328 90)
 			(effects
@@
 			)
 		)
-		(property "MPN" "RC0805FR-0743KL"
+		(property "MPN" "RC0603FR-0743KL"
 			(at 135.89 82.55 0)
 			(effects

Commit message: start layout
Parts:
- added C26: 1000pF, Capacitor_SMD:C_1206_3216Metric_Pad1.33x1.80mm_HandSolder, symbol Device:C_Small
Connections:
- net GND: now also C26.2
- net HV-Charger_out: now also C26.1
Other:
- moved on the sheet: J8
Changed lines of the file:
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@@
 	(text "Sektchy Spannungsmesser"
 		(exclude_from_sim no)
-		(at 186.69 97.79 0)
+		(at 193.04 97.79 0)
 		(effects
 			(font
@@
 	)
 	(junction
+		(at 180.34 69.85)
+		(diameter 0)
+		(color 0 0 0 0)
+	)
+	(junction
 		(at 72.39 69.85)
 		(diameter 0)
@@
 	)
 	(junction
-		(at 193.04 69.85)
+		(at 199.39 69.85)
 		(diameter 0)
 		(color 0 0 0 0)
 	)
 	(no_connect
-		(at 186.69 88.9)
+		(at 196.85 88.9)
 	)
 	(wire
@@
 	(wire
 		(pts
-			(xy 186.69 86.36) (xy 193.04 86.36)
+			(xy 196.85 86.36) (xy 199.39 86.36)
 		)
 		(stroke
@@
 	(wire
 		(pts
-			(xy 186.69 91.44) (xy 187.96 91.44)
+			(xy 196.85 91.44) (xy 198.12 91.44)
 		)
 		(stroke
@@
 	(wire
 		(pts
-			(xy 193.04 69.85) (xy 193.04 86.36)
+			(xy 199.39 69.85) (xy 199.39 86.36)
 		)
 		(stroke
@@
 	(wire
 		(pts
+			(xy 180.34 69.85) (xy 180.34 71.12)
+		)
+		(stroke
+			(width 0)
+			(type default)
+		)
+	)
+	(wire
+		(pts
 			(xy 82.55 69.85) (xy 82.55 71.12)
 		)
@@
 	(wire
 		(pts
+			(xy 180.34 76.2) (xy 180.34 77.47)
+		)
+		(stroke
+			(width 0)
+			(type default)
+		)
+	)
+	(wire
+		(pts
 			(xy 153.67 104.14) (xy 153.67 105.41)
 		)
@@
 	(wire
 		(pts
-			(xy 193.04 69.85) (xy 195.58 69.85)
+			(xy 199.39 69.85) (xy 201.93 69.85)
+		)
+		(stroke
+			(width 0)
+			(type default)
+		)
+	)
+	(wire
+		(pts
+			(xy 180.34 69.85) (xy 199.39 69.85)
 		)
 		(stroke
@@
 	(wire
 		(pts
-			(xy 186.69 93.98) (xy 187.96 93.98)
+			(xy 196.85 93.98) (xy 198.12 93.98)
 		)
 		(stroke
@@
 	(wire
 		(pts
-			(xy 81.28 87.63) (xy 82.55 87.63)
+			(xy 177.8 69.85) (xy 180.34 69.85)
 		)
 		(stroke
@@
 	(wire
 		(pts
-			(xy 144.78 88.9) (xy 144.78 87.63)
+			(xy 81.28 87.63) (xy 82.55 87.63)
 		)
 		(stroke
@@
 	(wire
 		(pts
-			(xy 72.39 71.12) (xy 72.39 69.85)
+			(xy 144.78 88.9) (xy 144.78 87.63)
 		)
 		(stroke
@@
 	(wire
 		(pts
-			(xy 130.81 107.95) (xy 130.81 109.22)
+			(xy 72.39 71.12) (xy 72.39 69.85)
 		)
 		(stroke
@@
 	(wire
 		(pts
-			(xy 130.81 64.77) (xy 118.11 64.77)
+			(xy 130.81 107.95) (xy 130.81 109.22)
 		)
 		(stroke
@@
 	(wire
 		(pts
-			(xy 177.8 69.85) (xy 193.04 69.85)
+			(xy 130.81 64.77) (xy 118.11 64.77)
 		)
 		(stroke
@@
 	(hierarchical_label "HV-Charger_out"
 		(shape output)
-		(at 195.58 69.85 0)
+		(at 201.93 69.85 0)
 		(effects
 			(font
@@
 	(symbol
 		(lib_id "power:GND")
-		(at 187.96 91.44 90)
+		(at 198.12 91.44 90)
 		(unit 1)
 		(exclude_from_sim no)
@@
 		(fields_autoplaced yes)
 		(property "Reference" "#PWR054"
-			(at 194.31 91.44 0)
+			(at 204.47 91.44 0)
 			(effects
 				(font
@@
 		)
 		(property "Value" "GND"
-			(at 191.77 91.4399 90)
+			(at 201.93 91.4399 90)
 			(effects
 				(font
@@
 		)
 		(property "Footprint" ""
-			(at 187.96 91.44 0)
+			(at 198.12 91.44 0)
 			(effects
 				(font
@@
 		)
 		(property "Datasheet" ""
-			(at 187.96 91.44 0)
+			(at 198.12 91.44 0)
 			(effects
 				(font
@@
 		)
 		(property "Description" "Power symbol creates a global label with name \"GND\" , ground"
-			(at 187.96 91.44 0)
+			(at 198.12 91.44 0)
 			(effects
 				(font
@@
 	(symbol
 		(lib_id "Connector_Generic:Conn_01x04")
-		(at 181.61 91.44 180)
+		(at 191.77 91.44 180)
 		(unit 1)
 		(exclude_from_sim no)
@@
 		(fields_autoplaced yes)
 		(property "Reference" "J8"
-			(at 181.61 80.01 0)
+			(at 191.77 80.01 0)
 			(effects
 				(font
@@
 		)
 		(property "Value" "Conn_01x04"
-			(at 181.61 82.55 0)
+			(at 191.77 82.55 0)
 			(effects
 				(font
@@
 		)
 		(property "Footprint" "Connector_PinHeader_2.54mm:PinHeader_1x04_P2.54mm_Vertical"
-			(at 181.61 91.44 0)
+			(at 191.77 91.44 0)
 			(effects
 				(font
@@
 		)
 		(property "Datasheet" "~"
-			(at 181.61 91.44 0)
+			(at 191.77 91.44 0)
 			(effects
 				(font
@@
 		)
 		(property "Description" "Generic connector, single row, 01x04, script generated (kicad-library-utils/schlib/autogen/connector/)"
-			(at 181.61 91.44 0)
+			(at 191.77 91.44 0)
 			(effects
 				(font
@@
 	(symbol
 		(lib_id "power:+5V")
-		(at 187.96 93.98 270)
+		(at 198.12 93.98 270)
 		(unit 1)
 		(exclude_from_sim no)
@@
 		(fields_autoplaced yes)
 		(property "Reference" "#PWR055"
-			(at 184.15 93.98 0)
+			(at 194.31 93.98 0)
 			(effects
 				(font
@@
 		)
 		(property "Value" "+5V"
-			(at 191.77 93.9799 90)
+			(at 201.93 93.9799 90)
 			(effects
 				(font
@@
 		)
 		(property "Footprint" ""
-			(at 187.96 93.98 0)
+			(at 198.12 93.98 0)
 			(effects
 				(font
@@
 		)
 		(property "Datasheet" ""
-			(at 187.96 93.98 0)
+			(at 198.12 93.98 0)
 			(effects
 				(font
@@
 		)
 		(property "Description" "Power symbol creates a global label with name \"+5V\""
-			(at 187.96 93.98 0)
+			(at 198.12 93.98 0)
 			(effects
 				(font
@@
 	)
 	(symbol
+		(lib_id "Device:C_Small")
+		(at 180.34 73.66 0)
+		(unit 1)
+		(exclude_from_sim no)
+		(in_bom yes)
+		(on_board yes)
+		(dnp no)
+		(property "Reference" "C26"
+			(at 181.61 71.12 0)
+			(effects
+				(font
+					(size 1.27 1.27)
+				)
+				(justify left)
+			)
+		)
+		(property "Value" "1000pF"
+			(at 181.61 76.2 0)
+			(effects
+				(font
+					(size 1.27 1.27)
+				)
+				(justify left)
+			)
+		)
+		(property "Footprint" "Capacitor_SMD:C_1206_3216Metric_Pad1.33x1.80mm_HandSolder"
+			(at 180.34 73.66 0)
+			(effects
+				(font
+					(size 1.27 1.27)
+				)
+				(hide yes)
+			)
+		)
+		(property "Datasheet" "~"
+			(at 180.34 73.66 0)
+			(effects
+				(font
+					(size 1.27 1.27)
+				)
+				(hide yes)
+			)
+		)
+		(property "Description" "Unpolarized capacitor, small symbol"
+			(at 180.34 73.66 0)
+			(effects
+				(font
+					(size 1.27 1.27)
+				)
+				(hide yes)
+			)
+		)
+		(property "MPN" "885342208018"
+			(at 180.34 73.66 0)
+			(effects
+				(font
+					(size 1.27 1.27)
+				)
+				(hide yes)
+			)
+		)
+		(property "Voltage" "1000V"
+			(at 180.34 73.66 0)
+			(effects
+				(font
+					(size 1.27 1.27)
+				)
+				(hide yes)
+			)
+		)
+		(pin "1"
+		)
+		(pin "2"
+		)
+		(instances
+			(project "Gaus-Beschleuniger"
+				(path "/10afecde-cced-4b16-9a8f-ba25affe517e/89601b47-33d3-45bd-90a7-6d36528e5bd8"
+					(reference "C26")
+					(unit 1)
+				)
+			)
+		)
+	)
+	(symbol
 		(lib_id "Device:R")
 		(at 143.51 77.47 90)
@@
 					(unit 1)
 				)
+			)
+		)
+	)
+	(symbol
+		(lib_id "power:GND")
+		(at 180.34 77.47 0)
+		(unit 1)
+		(exclude_from_sim no)
+		(in_bom yes)
+		(on_board yes)
+		(dnp no)
+		(fields_autoplaced yes)
+		(property "Reference" "#PWR067"
+			(at 180.34 83.82 0)
+			(effects
+				(font
+					(size 1.27 1.27)
+				)
+				(hide yes)
+			)
+		)
+		(property "Value" "GND"
+			(at 180.34 82.55 0)
+			(effects
+				(font
+					(size 1.27 1.27)
+				)
+			)
+		)
+		(property "Footprint" ""
+			(at 180.34 77.47 0)
+			(effects
+				(font
+					(size 1.27 1.27)
+				)
+				(hide yes)
+			)
+		)
+		(property "Datasheet" ""
+			(at 180.34 77.47 0)
+			(effects
+				(font
+					(size 1.27 1.27)
+				)
+				(hide yes)
+			)
+		)
+		(property "Description" "Power symbol creates a global label with name \"GND\" , ground"
+			(at 180.34 77.47 0)
+			(effects
+				(font
+					(size 1.27 1.27)
+				)
+				(hide yes)
+			)
+		)
+		(pin "1"
+		)
+		(instances
+			(project "Gaus-Beschleuniger"
+				(path "/10afecde-cced-4b16-9a8f-ba25affe517e/89601b47-33d3-45bd-90a7-6d36528e5bd8"
+					(reference "#PWR067")
+					(unit 1)
+				)

Commit message: update fab files ;/
Parts:
- C16, C17, C18, C19, C20, C21: LCSC_Part_# (none) -> C51205
- C22: LCSC_Part_# (none) -> C2167328
- C23, C24: LCSC_Part_# (none) -> C109392
- C26: LCSC_Part_# (none) -> C23631; MPN 885342208018 -> CC1206KKX7RDBB102
- D16: value 1000V -> US2M_HF; LCSC_Part_# (none) -> C17247425; Voltage (none) -> 1000V
- D18: LCSC_Part_# (none) -> C232444
- J8, J9: now not fitted
- Q9: LCSC_Part_# (none) -> C13914
- R26: LCSC_Part_# (none) -> C7023635
- R27: LCSC_Part_# (none) -> C137719
- R28: LCSC_Part_# (none) -> C4210186
- R29: LCSC_Part_# (none) -> C165742
- R30, R31: LCSC_Part_# (none) -> C84376
- U2: value ~ -> LT3750; LCSC_Part_# (none) -> C580129; MPN LT3750AEMS#TRPBF -> LT3750
Changed lines of the file:
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@@
 			)
 		)
-		(property "Value" "1000V"
+		(property "Value" "US2M_HF"
 			(at 173.99 66.04 0)
 			(effects
@@
 			)
 		)
+		(property "LCSC_Part_#" "C17247425"
+			(at 173.99 69.85 0)
+			(effects
+				(font
+					(size 1.27 1.27)
+				)
+				(hide yes)
+			)
+		)
+		(property "Voltage" "1000V"
+			(at 173.99 69.85 0)
+			(effects
+				(font
+					(size 1.27 1.27)
+				)
+				(hide yes)
+			)
+		)
 		(pin "2"
 		)
@@
 			)
 		)
+		(property "LCSC_Part_#" "C51205"
+			(at 62.23 86.36 0)
+			(effects
+				(font
+					(size 1.27 1.27)
+				)
+				(hide yes)
+			)
+		)
 		(pin "1"
 		)
@@
 		)
 		(property "MPN" "RC0805FR-0710KL"
+			(at 86.36 87.63 90)
+			(effects
+				(font
+					(size 1.27 1.27)
+				)
+				(hide yes)
+			)
+		)
+		(property "LCSC_Part_#" "C84376"
 			(at 86.36 87.63 90)
 			(effects
@@
 			)
 		)
+		(property "LCSC_Part_#" "C4210186"
+			(at 130.81 104.14 0)
+			(effects
+				(font
+					(size 1.27 1.27)
+				)
+				(hide yes)
+			)
+		)
 		(pin "1"
 		)
@@
 			)
 		)
+		(property "LCSC_Part_#" "C109392"
+			(at 130.81 68.58 0)
+			(effects
+				(font
+					(size 1.27 1.27)
+				)
+				(hide yes)
+			)
+		)
 		(pin "1"
 		)
@@
 		(in_bom yes)
 		(on_board yes)
-		(dnp no)
+		(dnp yes)
 		(fields_autoplaced yes)
 		(property "Reference" "J8"
@@
 			)
 		)
+		(property "LCSC_Part_#" ""
+			(at 191.77 91.44 0)
+			(effects
+				(font
+					(size 1.27 1.27)
+				)
+				(hide yes)
+			)
+		)
 		(pin "2"
 		)
@@
 		)
 		(property "Voltage" "50V"
+			(at 67.31 86.36 0)
+			(effects
+				(font
+					(size 1.27 1.27)
+				)
+				(hide yes)
+			)
+		)
+		(property "LCSC_Part_#" "C51205"
 			(at 67.31 86.36 0)
 			(effects
@@
 			)
 		)
+		(property "LCSC_Part_#" ""
+			(at 161.29 72.39 0)
+			(effects
+				(font
+					(size 1.27 1.27)
+				)
+				(hide yes)
+			)
+		)
 		(pin "6"
 		)
@@
 		(in_bom yes)
 		(on_board yes)
-		(dnp no)
+		(dnp yes)
 		(fields_autoplaced yes)
 		(property "Reference" "J9"
@@
 			)
 		)
+		(property "LCSC_Part_#" ""
+			(at 30.48 69.85 0)
+			(effects
+				(font
+					(size 1.27 1.27)
+				)
+				(hide yes)
+			)
+		)
 		(pin "3"
 		)
@@
 			)
 		)
+		(property "LCSC_Part_#" "C7023635"
+			(at 153.67 100.33 0)
+			(effects
+				(font
+					(size 1.27 1.27)
+				)
+				(hide yes)
+			)
+		)
 		(pin "1"
 		)
@@
 		)
 		(property "Voltage" "50V"
+			(at 140.97 104.14 0)
+			(effects
+				(font
+					(size 1.27 1.27)
+				)
+				(hide yes)
+			)
+		)
+		(property "LCSC_Part_#" "C2167328"
 			(at 140.97 104.14 0)
 			(effects
@@
 			)
 		)
+		(property "LCSC_Part_#" "C232444"
+			(at 40.64 76.2 90)
+			(effects
+				(font
+					(size 1.27 1.27)
+				)
+				(hide yes)
+			)
+		)
 		(pin "2"
 		)
@@
 			)
 		)
+		(property "LCSC_Part_#" "C84376"
+			(at 99.06 100.33 0)
+			(effects
+				(font
+					(size 1.27 1.27)
+				)
+				(hide yes)
+			)
+		)
 		(pin "2"
 		)
@@
 		)
 		(property "MPN" "35ZLH100MEFC6.3X11"
+			(at 118.11 68.58 0)
+			(effects
+				(font
+					(size 1.27 1.27)
+				)
+				(hide yes)
+			)
+		)
+		(property "LCSC_Part_#" "C109392"
 			(at 118.11 68.58 0)
 			(effects
@@
 			)
 		)
-		(property "MPN" "885342208018"
+		(property "MPN" "CC1206KKX7RDBB102"
 			(at 180.34 73.66 0)
 			(effects
@@
 		)
 		(property "Voltage" "1000V"
+			(at 180.34 73.66 0)
+			(effects
+				(font
+					(size 1.27 1.27)
+				)
+				(hide yes)
+			)
+		)
+		(property "LCSC_Part_#" "C23631"
 			(at 180.34 73.66 0)
 			(effects
@@
 			)
 		)
+		(property "LCSC_Part_#" "C165742"
+			(at 143.51 77.47 90)
+			(effects
+				(font
+					(size 1.27 1.27)
+				)
+				(hide yes)
+			)
+		)
 		(pin "2"
 		)
@@
 			)
 		)
-		(property "Value" "~"
+		(property "Value" "LT3750"
 			(at 117.348 69.85 0)
 			(effects
@@
 			)
 		)
-		(property "MPN" "LT3750AEMS#TRPBF"
+		(property "MPN" "LT3750"
+			(at 115.57 87.63 0)
+			(effects
+				(font
+					(size 1.27 1.27)
+				)
+				(hide yes)
+			)
+		)
+		(property "LCSC_Part_#" "C580129"
 			(at 115.57 87.63 0)
 			(effects
@@
 		)
 		(property "Voltage" "50V"
+			(at 77.47 73.66 0)
+			(effects
+				(font
+					(size 1.27 1.27)
+				)
+				(hide yes)
+			)
+		)
+		(property "LCSC_Part_#" "C51205"
 			(at 77.47 73.66 0)
 			(effects
@@
 			)
 		)
+		(property "LCSC_Part_#" "C13914"
+			(at 151.13 88.9 0)
+			(effects
+				(font
+					(size 1.27 1.27)
+				)
+				(hide yes)
+			)
+		)
 		(pin "5"
 		)
@@
 			)
 		)
+		(property "LCSC_Part_#" ""
+			(at 95.25 87.63 0)
+			(effects
+				(font
+					(size 1.27 1.27)
+				)
+				(hide yes)
+			)
+		)
 		(pin "1"
 		)
@@
 			)
 		)
+		(property "LCSC_Part_#" "C51205"
+			(at 57.15 86.36 0)
+			(effects
+				(font
+					(size 1.27 1.27)
+				)
+				(hide yes)
+			)
+		)
 		(pin "1"
 		)
@@
 			)
 		)
+		(property "LCSC_Part_#" "C51205"
+			(at 72.39 73.66 0)
+			(effects
+				(font
+					(size 1.27 1.27)
+				)
+				(hide yes)
+			)
+		)
 		(pin "1"
 		)
@@
 		)
 		(property "Voltage" "50V"
+			(at 82.55 73.66 0)
+			(effects
+				(font
+					(size 1.27 1.27)
+				)
+				(hide yes)
+			)
+		)
+		(property "LCSC_Part_#" "C51205"
 			(at 82.55 73.66 0)
 			(effects
@@
 			(effects
 				(font
+					(size 1.27 1.27)
+				)
+				(hide yes)
+			)
+		)
+		(property "LCSC_Part_#" "C137719"
+			(at 135.89 82.55 90)
+			(effects
+				(font
