File: Firing-Stage.kicad_sch (KiCad schematic)
At the start: 56 parts, among them J1 Conn_01x02, J2 Conn_01x02, J3 Conn_01x02, J4 Conn_01x02, J5 Conn_01x02, J6 Conn_01x02, Q1 Q_NMOS_GDS, Q2 Q_NMOS_GDS, Q3 940nm, Q4 940nm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

Commit message: rough placement
Parts:
- C1, C2, C3, C4, C5, C6, C7, C8: value 330u -> 1000uF; footprint (none) -> Capacitor_THT:CP_Radial_D35.0mm_P10.00mm_SnapIn; MPN (none) -> ESMR401VSN102MA50S
- R10, R11, R13, R15, R17, R20, R21, R22, R24, R3, R6, R7: MPN (none) -> RC0805FR-0710KL
- R12, R14, R16, R5: MPN (none) -> RC0805FR-101KL
- R18, R19, R4, R9: MPN (none) -> RNV14FAL470K
- R23, R8: MPN (none) -> SQP10AJB-2K

Commit message: start layout
Parts:
- removed D23: D_Schottky, Diode_SMD:D_SOD-123, symbol Device:D_Schottky
- removed R21, R22: 10k, Resistor_SMD:R_0805_2012Metric_Pad1.20x1.40mm_HandSolder, symbol Device:R
- D15, D4: footprint Package_TO_SOT_THT:TO-247-3_Vertical -> Package_TO_SOT_THT:TO-247-3_Horizontal_TabDown
- Q3, Q4, Q5, Q6: footprint LED_THT:LED_SideEmitter_Rectangular_W4.5mm_H1.6mm -> OptoDevice:Osram_LPT80A
Connections:
- net HV_S1: no longer J4.1 (Pin_1), J4.2 (Pin_2)
- net HV_S2: now also J4.1 (Pin_1), J4.2 (Pin_2)
- net discharge_gate: now reaches Q2.1 (G)
- net discharge_gate: now also D24.1 (K), Q1.1 (G), R6.1, R7.2

Commit message: layout weiter
Connections:
- net S2_D: now reaches D15.2 (A), J6.2 (Pin_2)
- net S1_D: now reaches D4.2 (A), J1.2 (Pin_2)
Changed lines of the file:
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@@
+		)
+	)
+	(label "S2_D"
+		(at 165.1 118.11 0)
+		(effects
+			(font
+				(size 1.27 1.27)
+			)
+			(justify left bottom)
 		)
 	)
@@
 		)
 	)
+	(label "S1_D"
+		(at 165.1 59.69 0)
+		(effects
+			(font
+				(size 1.27 1.27)
+			)
+			(justify left bottom)
+		)
+	)

Commit message: update fab files ;/
Parts:
- C1, C2, C3, C4, C5, C6, C7, C8: LCSC_Part_# (none) -> C1589731
- D10, D12, D7, D8: LCSC_Part_# (none) -> C6980548
- D15, D4: LCSC_Part_# (none) -> C335786
- D24: LCSC_Part_# (none) -> C154764
- D25, D5: LCSC_Part_# (none) -> C16378
- Q3, Q4, Q5, Q6: LCSC_Part_# (none) -> C17179478
- R10, R11, R13, R15, R17, R20, R24, R3, R6, R7: LCSC_Part_# (none) -> C84376
- R12, R14, R16, R5: LCSC_Part_# (none) -> C5842544
- R18, R19, R4, R9: LCSC_Part_# (none) -> C2642472
- R23, R8: value 2k 5W SQP10AJB-2K -> 2k; LCSC_Part_# (none) -> C20166277
